File: Power strip/XPNET hub.sch (EAGLE design)
At the start: 16 parts, among them X1 MKDSN1,5/4-5,08, X4 MKDSN1,5/4-5,08, X5 MKDSN1,5/4-5,08, X6 MKDSN1,5/4-5,08

Commit message: Add files via upload
Parts:
- removed LED2, LED3: Blue, adafruit:LED3MM
- removed LOGO1: OSHW_LOGO_6MILX0200-NT, ohw-logo:OSHW_LOGO_6MILX0200-NT
- removed X2, X3: (no value), con-phoenix-500:MSTBV8
- removed X4, X5, X6: MKDSN1,5/4-5,08, con-phoenix-508:MKDSN1,5/4-5,08
- added D1, D2: VISHAY_SCHOTTKY, Ava:VISHAY_SCHOTTKY
- added J1, J2, J3, J4, J5, J6: RJ11-6SMALL, GJR:RJ11-6SMALL
- added LED4: Green, adafruit:LED3MM
- LED1: value WHITE -> Green
- X1: value MKDSN1,5/4-5,08 -> 1751264; device con-phoenix-508:MKDSN1,5/4-5,08 -> con-phoenix-350:1751264
Connections:
- removed net +15V: LED3.A, X1-3.KL, X4-3.KL, X5-3.KL, X6-3.KL
- removed net DCC1: LED1.A, LED2.C, X1-1.KL, X2-2.SK, X2-4.SK, X2-6.SK, X2-8.SK, X3-2.SK, X3-4.SK, X3-6.SK, X3-8.SK, X4-1.KL, X5-1.KL, X6-1.KL
- removed net DCC2: R1.1, X1-2.KL, X2-1.SK, X2-3.SK, X2-5.SK, X2-7.SK, X3-1.SK, X3-3.SK, X3-5.SK, X3-7.SK, X4-2.KL, X5-2.KL, X6-2.KL
- removed net N$32: LED1.C, LED2.A, R1.2
- new net +12V: D1.C, D2.C, J2.5, J3.5, J4.5, J5.5, J6.5
- new net +21V1: D2.A, LED1.A, X1-4.K
- new net A: J1.4, J2.4, J3.4, J4.4, J5.4, J6.4, X1-2.K
- new net B: J1.3, J2.3, J3.3, J4.3, J5.3, J6.3, X1-3.K
- new net CMD_ACK: J1.6, J2.6, J3.6, J4.6, J5.6, J6.6
- new net GND_RTN: J1.1, J2.1, J3.1, J4.1, J5.1, J6.1
- new net N$19: LED4.C, R2.2
- new net N$3: LED1.C, R1.2
- net GND: now also J1.2, J2.2, J3.2, J4.2, J5.2, J6.2, R1.1, X1-1.K; no longer X1-4.KL, X4-4.KL, X5-4.KL, X6-4.KL
- net N$1: now also D1.A, J1.5, LED4.A; no longer LED3.C, R2.2
Other:
- moved on the sheet: H1, H2, H3, H4, LED1, R1, R2
